File: vgaterm-io/vgaterm-io.kicad_sch (KiCad schematic)
At the start: 32 parts, among them J1 Conn_01x04, J2 Conn_01x04, J4 DE9_Receptacle, J5 Conn_02x08_Top_Bottom Switch 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, J6 USB_B_Micro Debug, J7 RJ45_LED, J8 Conn_01x10 Data Conn, Q1 Q_Dual_PMOS_S1G1D2S2G2D1, Q2 Q_Dual_PMOS_S1G1D2S2G2D1, Q3 Q_Dual_PMOS_S1G1D2S2G2D1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

Commit message: updating board based on convos with Seth
Parts:
- R11, R12, R15, R16, R7, R8: value 20k -> 40k
- R3, R4: value 20k -> 300k
Changed lines of the file:
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@@
       (effects (font (size 1.27 1.27)))
     )
-    (property "Value" "20k" (at 124.46 165.1 90)
+    (property "Value" "40k" (at 124.46 165.1 90)
       (effects (font (size 1.27 1.27)))
     )
@@
       (effects (font (size 1.27 1.27)))
     )
-    (property "Value" "20k" (at 124.46 181.61 90)
+    (property "Value" "40k" (at 124.46 181.61 90)
       (effects (font (size 1.27 1.27)))
     )
@@
       (effects (font (size 1.27 1.27)))
     )
-    (property "Value" "20k" (at 128.27 57.15 90)
+    (property "Value" "300k" (at 128.27 57.15 90)
       (effects (font (size 1.27 1.27)))
     )
@@
       (effects (font (size 1.27 1.27)))
     )
-    (property "Value" "20k" (at 125.73 85.09 90)
+    (property "Value" "40k" (at 125.73 85.09 90)
       (effects (font (size 1.27 1.27)))
     )
@@
       (effects (font (size 1.27 1.27)))
     )
-    (property "Value" "20k" (at 125.73 124.46 90)
+    (property "Value" "40k" (at 125.73 124.46 90)
       (effects (font (size 1.27 1.27)))
     )
@@
       (effects (font (size 1.27 1.27)))
     )
-    (property "Value" "20k" (at 125.73 140.97 90)
+    (property "Value" "40k" (at 125.73 140.97 90)
       (effects (font (size 1.27 1.27)))
     )
@@
       (effects (font (size 1.27 1.27)))
     )
-    (property "Value" "20k" (at 128.27 40.64 90)
+    (property "Value" "300k" (at 128.27 40.64 90)
       (effects (font (size 1.27 1.27)))
     )
@@
       (effects (font (size 1.27 1.27)))
     )
-    (property "Value" "20k" (at 125.73 101.6 90)
-      (effects (font (size 1.27 1.27)))
-    )
+    (property "Value" "40k" (at 125.73 101.6 90)
+      (effects (font (size 1.27 1.27)))
+    )
