File: vgaterm-schematics.kicad_sch (KiCad schematic)
At the start: 23 parts, among them J1 Conn_01x04, J1 Conn_01x15, J1 Conn_01x15_Socket, J4 Conn_01x15_Socket, J6 Conn_01x03_Socket, J6 Conn_01x10, U1 GAL22V10, U2 74HCT574, U3 74AHCT244, U4 IDT7205L12JG

Commit message: updating board based on convos with Seth
Parts:
- added J2: Rst, Connector_PinHeader_2.54mm:PinHeader_1x02_P2.54mm_Vertical, symbol Connector_Generic:Conn_01x02
- added R2: R, Resistor_SMD:R_0805_2012Metric_Pad1.20x1.40mm_HandSolder, symbol Device:R
Connections:
- net GND: now also J2.1 (Pin_1)
- net VCC: now also R2.2
- net Rst: now reaches J1.4 (Pin_4)
- net Rst: now also J2.2 (Pin_2), R2.1
- no-connect marks 10 -> 9
Changed lines of the file:
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@@
   (junction (at 54.61 35.56) (diameter 0) (color 0 0 0 0)
+  )
+  (junction (at 29.21 21.59) (diameter 0) (color 0 0 0 0)
   )
   (junction (at 85.09 111.76) (diameter 0) (color 0 0 0 0)
@@
   (no_connect (at 26.67 35.56))
   (no_connect (at 167.64 132.08))
-  (no_connect (at 31.75 35.56))
   (no_connect (at 172.72 81.28))
   (no_connect (at 52.07 35.56))
@@
     (stroke (width 0) (type default))
   )
+  (wire (pts (xy 29.21 21.59) (xy 29.21 25.4))
+    (stroke (width 0) (type default))
+  )
   (wire (pts (xy 41.91 86.36) (xy 46.99 86.36))
     (stroke (width 0) (type default))
@@
     (effects (font (size 1.27 1.27)) (justify right bottom))
   )
+  (label "Rst" (at 31.75 35.56 270) (fields_autoplaced)
+    (effects (font (size 1.27 1.27)) (justify right bottom))
+  )
   (label "DO+" (at 41.91 140.97 90) (fields_autoplaced)
     (effects (font (size 1.27 1.27)) (justify left bottom))
@@
     (effects (font (size 1.27 1.27)) (justify right bottom))
   )
+  (label "Rst" (at 29.21 25.4 0) (fields_autoplaced)
+    (effects (font (size 1.27 1.27)) (justify left bottom))
+  )
   (label "P7" (at 262.89 120.65 0) (fields_autoplaced)
     (effects (font (size 1.27 1.27)) (justify left bottom))
@@
         (path "/6b101ec3-37f4-4299-ac87-721c8a68e9ce"
           (reference "#PWR036") (unit 1)
+        )
+      )
+    )
+  )
+  (symbol (lib_id "power:VCC") (at 36.83 21.59 270) (unit 1)
+    (in_bom yes) (on_board yes) (dnp no) (fields_autoplaced)
+    (property "Reference" "#PWR011" (at 33.02 21.59 0)
+      (effects (font (size 1.27 1.27)) hide)
+    )
+    (property "Value" "VCC" (at 40.64 21.5899 90)
+      (effects (font (size 1.27 1.27)) (justify left))
+    )
+    (property "Footprint" "" (at 36.83 21.59 0)
+      (effects (font (size 1.27 1.27)) hide)
+    )
+    (property "Datasheet" "" (at 36.83 21.59 0)
+      (effects (font (size 1.27 1.27)) hide)
+    )
+    (pin "1")
+    (instances
+      (project "cpu_data"
+        (path "/56a776f8-148b-473a-851d-f1ac7e6b3eea"
+          (reference "#PWR011") (unit 1)
+        )
+      )
+      (project "vgaterm-schematics"
+        (path "/6b101ec3-37f4-4299-ac87-721c8a68e9ce"
+          (reference "#PWR06") (unit 1)
         )
       )
@@
     )
   )
+  (symbol (lib_id "Connector_Generic:Conn_01x02") (at 26.67 16.51 90) (unit 1)
+    (in_bom yes) (on_board yes) (dnp no) (fields_autoplaced)
+    (property "Reference" "J2" (at 31.75 15.24 90)
+      (effects (font (size 1.27 1.27)) (justify right))
+    )
+    (property "Value" "Rst" (at 31.75 17.78 90)
+      (effects (font (size 1.27 1.27)) (justify right))
+    )
+    (property "Footprint" "Connector_PinHeader_2.54mm:PinHeader_1x02_P2.54mm_Vertical" (at 26.67 16.51 0)
+      (effects (font (size 1.27 1.27)) hide)
+    )
+    (property "Datasheet" "~" (at 26.67 16.51 0)
+      (effects (font (size 1.27 1.27)) hide)
+    )
+    (pin "1")
+    (pin "2")
+    (instances
+      (project "vgaterm-schematics"
+        (path "/6b101ec3-37f4-4299-ac87-721c8a68e9ce"
+          (reference "J2") (unit 1)
+        )
+      )
+    )
+  )
   (symbol (lib_id "Connector:Conn_01x15_Socket") (at 41.91 30.48 90) (unit 1)
     (in_bom yes) (on_board yes) (dnp no) (fields_autoplaced)
@@
     )
   )
+  (symbol (lib_id "power:GND") (at 26.67 21.59 0) (unit 1)
+    (in_bom yes) (on_board yes) (dnp no) (fields_autoplaced)
+    (property "Reference" "#PWR01" (at 26.67 27.94 0)
+      (effects (font (size 1.27 1.27)) hide)
+    )
+    (property "Value" "GND" (at 26.67 26.67 0)
+      (effects (font (size 1.27 1.27)))
+    )
+    (property "Footprint" "" (at 26.67 21.59 0)
+      (effects (font (size 1.27 1.27)) hide)
+    )
+    (property "Datasheet" "" (at 26.67 21.59 0)
+      (effects (font (size 1.27 1.27)) hide)
+    )
+    (pin "1")
+    (instances
+      (project "cpu_data"
+        (path "/56a776f8-148b-473a-851d-f1ac7e6b3eea"
+          (reference "#PWR01") (unit 1)
+        )
+      )
+      (project "vgaterm-schematics"
+        (path "/6b101ec3-37f4-4299-ac87-721c8a68e9ce"
+          (reference "#PWR07") (unit 1)
+        )
+      )
+    )
+  )
   (symbol (lib_id "Device:C_Small") (at 53.34 80.01 90) (unit 1)
     (in_bom yes) (on_board yes) (dnp no) (fields_autoplaced)
@@
         )
       )
+    )
+  )
+  (symbol (lib_id "Device:R") (at 33.02 21.59 90) (unit 1)
+    (in_bom yes) (on_board yes) (dnp no) (fields_autoplaced)
+    (property "Reference" "R2" (at 33.02 15.24 90)
+      (effects (font (size 1.27 1.27)))
+    )
+    (property "Value" "R" (at 33.02 17.78 90)
+      (effects (font (size 1.27 1.27)))
+    )
+    (property "Footprint" "Resistor_SMD:R_0805_2012Metric_Pad1.20x1.40mm_HandSolder" (at 33.02 23.368 90)
+      (effects (font (size 1.27 1.27)) hide)
+    )
+    (property "Datasheet" "~" (at 33.02 21.59 0)
+      (effects (font (size 1.27 1.27)) hide)
+    )
+    (pin "1")
+    (pin "2")
+    (instances
+      (project "vgaterm-schematics"
+        (path "/6b101ec3-37f4-4299-ac87-721c8a68e9ce"
+          (reference "R2") (unit 1)
+        )
+      )

Commit message: current boards
Parts:
- added C6: 220n, Capacitor_SMD:C_0805_2012Metric_Pad1.18x1.45mm_HandSolder, symbol Device:C_Small
- added R3: 330, Resistor_SMD:R_0805_2012Metric_Pad1.20x1.40mm_HandSolder, symbol Device:R
Connections:
- net Clk_{pixel}: now also R3.1
- net GND: now also C6.2
- new net: C6.1, R3.2
Changed lines of the file:
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@@
+    (effects (font (size 1.27 1.27)) (justify right bottom))
+  )
+  (label "Clk_{pixel}" (at 73.66 66.04 180) (fields_autoplaced)
     (effects (font (size 1.27 1.27)) (justify right bottom))
   )
@@
     )
   )
+  (symbol (lib_id "Device:C_Small") (at 83.82 66.04 90) (unit 1)
+    (in_bom yes) (on_board yes) (dnp no) (fields_autoplaced)
+    (property "Reference" "C6" (at 83.8263 59.69 90)
+      (effects (font (size 1.27 1.27)))
+    )
+    (property "Value" "220n" (at 83.8263 62.23 90)
+      (effects (font (size 1.27 1.27)))
+    )
+    (property "Footprint" "Capacitor_SMD:C_0805_2012Metric_Pad1.18x1.45mm_HandSolder" (at 83.82 66.04 0)
+      (effects (font (size 1.27 1.27)) hide)
+    )
+    (property "Datasheet" "~" (at 83.82 66.04 0)
+      (effects (font (size 1.27 1.27)) hide)
+    )
+    (pin "2")
+    (pin "1")
+    (instances
+      (project "vgaterm-schematics"
+        (path "/6b101ec3-37f4-4299-ac87-721c8a68e9ce"
+          (reference "C6") (unit 1)
+        )
+      )
+    )
+  )
   (symbol (lib_id "power:GND") (at 39.37 105.41 270) (unit 1)
     (in_bom yes) (on_board yes) (dnp no) (fields_autoplaced)
@@
         (path "/6b101ec3-37f4-4299-ac87-721c8a68e9ce"
           (reference "#FLG01") (unit 1)
+        )
+      )
+    )
+  )
+  (symbol (lib_id "Device:R") (at 77.47 66.04 90) (unit 1)
+    (in_bom yes) (on_board yes) (dnp no) (fields_autoplaced)
+    (property "Reference" "R3" (at 77.47 59.69 90)
+      (effects (font (size 1.27 1.27)))
+    )
+    (property "Value" "330" (at 77.47 62.23 90)
+      (effects (font (size 1.27 1.27)))
+    )
+    (property "Footprint" "Resistor_SMD:R_0805_2012Metric_Pad1.20x1.40mm_HandSolder" (at 77.47 67.818 90)
+      (effects (font (size 1.27 1.27)) hide)
+    )
+    (property "Datasheet" "~" (at 77.47 66.04 0)
+      (effects (font (size 1.27 1.27)) hide)
+    )
+    (pin "2")
+    (pin "1")
+    (instances
+      (project "vgaterm-schematics"
+        (path "/6b101ec3-37f4-4299-ac87-721c8a68e9ce"
+          (reference "R3") (unit 1)
         )
       )
@@
         )
       )
+    )
+  )
+  (symbol (lib_id "power:GND") (at 86.36 66.04 0) (unit 1)
+    (in_bom yes) (on_board yes) (dnp no) (fields_autoplaced)
+    (property "Reference" "#PWR033" (at 86.36 72.39 0)
+      (effects (font (size 1.27 1.27)) hide)
+    )
+    (property "Value" "GND" (at 86.36 71.12 0)
+      (effects (font (size 1.27 1.27)))
+    )
+    (property "Footprint" "" (at 86.36 66.04 0)
+      (effects (font (size 1.27 1.27)) hide)
+    )
+    (property "Datasheet" "" (at 86.36 66.04 0)
+      (effects (font (size 1.27 1.27)) hide)
+    )
+    (pin "1")
+    (instances
+      (project "vgaterm-schematics"
+        (path "/6b101ec3-37f4-4299-ac87-721c8a68e9ce"
+          (reference "#PWR033") (unit 1)
+        )
+      )
