File: keyboard-loft/keyboard-loft.kicad_sch (KiCad schematic)
At the start: 2 parts, among them J1 Conn_01x04

Commit message: current boards
Parts:
- added H1 (x2): MountingHole, MountingHole:MountingHole_2.2mm_M2_ISO7380, symbol Mechanical:MountingHole
- J1: footprint Connector_PinHeader_2.54mm:PinHeader_2x02_P2.54mm_Vertical_SMD -> Connector_PinHeader_2.54mm:PinHeader_1x04_P2.54mm_Horizontal
Changed lines of the file:
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@@
       (effects (font (size 1.27 1.27)) (justify left))
     )
-    (property "Footprint" "Connector_PinHeader_2.54mm:PinHeader_2x02_P2.54mm_Vertical_SMD" (at 113.03 86.36 0)
+    (property "Footprint" "Connector_PinHeader_2.54mm:PinHeader_1x04_P2.54mm_Horizontal" (at 113.03 86.36 0)
       (effects (font (size 1.27 1.27)) hide)
     )
@@
         )
       )
+    )
+  )
+  (symbol (lib_id "Mechanical:MountingHole") (at 120.65 68.58 0) (unit 1)
+    (in_bom yes) (on_board yes) (dnp no) (fields_autoplaced)
+    (property "Reference" "H1" (at 123.19 67.31 0)
+      (effects (font (size 1.27 1.27)) (justify left))
+    )
+    (property "Value" "MountingHole" (at 123.19 69.85 0)
+      (effects (font (size 1.27 1.27)) (justify left))
+    )
+    (property "Footprint" "MountingHole:MountingHole_2.2mm_M2_ISO7380" (at 120.65 68.58 0)
+      (effects (font (size 1.27 1.27)) hide)
+    )
+    (property "Datasheet" "~" (at 120.65 68.58 0)
+      (effects (font (size 1.27 1.27)) hide)
+    )
+    (instances
+      (project "vgaterm-bottom"
+        (path "/0bae2297-ffc0-4205-a707-96188a2849e2"
+          (reference "H1") (unit 1)
+        )
+      )
+      (project "vgaterm-io"
+        (path "/94313e75-2556-4a4f-b866-652a05fdde62"
+          (reference "H1") (unit 1)
+        )
+      )
+      (project "keyboard-loft"
+        (path "/9c23afe2-e8ac-4f84-b3d7-40da52448ecc"
+          (reference "H2") (unit 1)
+        )
+      )
+    )
+  )
+  (symbol (lib_id "Mechanical:MountingHole") (at 101.6 68.58 0) (unit 1)
+    (in_bom yes) (on_board yes) (dnp no) (fields_autoplaced)
+    (property "Reference" "H1" (at 104.14 67.31 0)
+      (effects (font (size 1.27 1.27)) (justify left))
+    )
+    (property "Value" "MountingHole" (at 104.14 69.85 0)
+      (effects (font (size 1.27 1.27)) (justify left))
+    )
+    (property "Footprint" "MountingHole:MountingHole_2.2mm_M2_ISO7380" (at 101.6 68.58 0)
+      (effects (font (size 1.27 1.27)) hide)
+    )
+    (property "Datasheet" "~" (at 101.6 68.58 0)
+      (effects (font (size 1.27 1.27)) hide)
+    )
+    (instances
+      (project "vgaterm-bottom"
+        (path "/0bae2297-ffc0-4205-a707-96188a2849e2"
+          (reference "H1") (unit 1)
+        )
+      )
+      (project "vgaterm-io"
+        (path "/94313e75-2556-4a4f-b866-652a05fdde62"
+          (reference "H1") (unit 1)
+        )
+      )
+      (project "keyboard-loft"
+        (path "/9c23afe2-e8ac-4f84-b3d7-40da52448ecc"
+          (reference "H1") (unit 1)
+        )
+      )
