File: vga-breakout/vga-breakout.kicad_pcb (KiCad board)
At the start: 2 copper layers, 31.2 x 19.8 mm, 2 parts, among them J1 DE15_Receptacle_HighDensity_M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, J2 Conn_01x09

Commit message: current boards
Parts:
- J1: footprint Connector_Dsub:DSUB-15-HD_Female_Horizontal_P2.29x1.98mm_EdgePinOffset8.35mm_Housed_MountingHolesOffset10.89mm -> local:DSUB-15-HD_Female_Horizontal_P2.29x2.54mm_EdgePinOffset8.35mm_Housed_MountingHolesOffset10.89mm
- moved J1 1.51 mm to (144.6, 66.8)
Routing:
- net GND: track 4.22 -> 0.00 mm
- net /GND_{green}: track 8.57 -> 10.6 mm
- net /GND_{blue}: track 7.83 -> 9.90 mm
- net /HSYNC: track 20.6 -> 22.2 mm
- net /VSYNC: track 16.5 -> 18.1 mm
- net /Red: track 7.16 -> 8.68 mm
- net /Green: track 6.01 -> 7.52 mm
- net /Blue: track 6.43 -> 7.94 mm
- net /GND_{red}: track 10.5 -> 11.8 mm
Other:
- board size 31.2 x 19.8 mm -> 31.2 x 17.5 mm
