File: vga-breakout/vga-breakout.kicad_sch (KiCad schematic)
At the start: 2 parts, among them J2 Conn_01x09, J3 DE15_Receptacle_HighDensity_M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

Commit message: timing board updates and adding keyboard loft board and vga breakout
Parts:
- J2: footprint (none) -> Connector_PinHeader_2.54mm:PinHeader_1x09_P2.54mm_Vertical
Changed lines of the file:
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@@
     (effects (font (size 1.27 1.27)) (justify left bottom))
+  )
+  (symbol (lib_id "power:PWR_FLAG") (at 186.69 73.66 0) (unit 1)
+    (in_bom yes) (on_board yes) (dnp no) (fields_autoplaced)
+    (property "Reference" "#FLG01" (at 186.69 71.755 0)
+      (effects (font (size 1.27 1.27)) hide)
+    )
+    (property "Value" "PWR_FLAG" (at 186.69 68.58 0)
+      (effects (font (size 1.27 1.27)))
+    )
+    (property "Footprint" "" (at 186.69 73.66 0)
+      (effects (font (size 1.27 1.27)) hide)
+    )
+    (property "Datasheet" "~" (at 186.69 73.66 0)
+      (effects (font (size 1.27 1.27)) hide)
+    )
+    (pin "1")
+    (instances
+      (project "vga-breakout"
+        (path "/7e90bbd9-a941-471e-89d1-7a93f3ff40c6"
+          (reference "#FLG01") (unit 1)
+        )
+      )
+    )
   )
   (symbol (lib_id "power:GND") (at 153.67 74.93 0) (unit 1)
@@
       (effects (font (size 1.27 1.27)))
     )
-    (property "Footprint" "" (at 146.05 105.41 0)
+    (property "Footprint" "Connector_PinHeader_2.54mm:PinHeader_1x09_P2.54mm_Vertical" (at 146.05 105.41 0)
       (effects (font (size 1.27 1.27)) hide)
     )
@@
         )
       )
+    )
+  )
+  (symbol (lib_id "power:GND") (at 186.69 73.66 0) (unit 1)
+    (in_bom yes) (on_board yes) (dnp no) (fields_autoplaced)
+    (property "Reference" "#PWR048" (at 186.69 80.01 0)
+      (effects (font (size 1.27 1.27)) hide)
+    )
+    (property "Value" "GND" (at 186.69 78.74 0)
+      (effects (font (size 1.27 1.27)))
+    )
+    (property "Footprint" "" (at 186.69 73.66 0)
+      (effects (font (size 1.27 1.27)) hide)
+    )
+    (property "Datasheet" "" (at 186.69 73.66 0)
+      (effects (font (size 1.27 1.27)) hide)
+    )
+    (pin "1")
+    (instances
+      (project "vgaterm-timing-vga"
+        (path "/2507db06-1687-4aca-8562-74daa0e6a71c"
+          (reference "#PWR048") (unit 1)
+        )
+      )
+      (project "vga-breakout"
+        (path "/7e90bbd9-a941-471e-89d1-7a93f3ff40c6"
+          (reference "#PWR02") (unit 1)
+        )
+      )
+      (project "vga-connection"
+        (path "/96e66b69-8426-4b51-b32a-8435b751d1a6"
+          (reference "#PWR019") (unit 1)
+        )
+      )

Commit message: current boards
Parts:
- J3: footprint Connector_Dsub:DSUB-15-HD_Female_Horizontal_P2.29x1.98mm_EdgePinOffset8.35mm_Housed_MountingHolesOffset10.89mm -> local:DSUB-15-HD_Female_Horizontal_P2.29x2.54mm_EdgePinOffset8.35mm_Housed_MountingHolesOffset10.89mm
Changed lines of the file:
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@@
       (effects (font (size 1.27 1.27)) (justify left))
     )
-    (property "Footprint" "Connector_Dsub:DSUB-15-HD_Female_Horizontal_P2.29x1.98mm_EdgePinOffset8.35mm_Housed_MountingHolesOffset10.89mm" (at 133.35 91.44 0)
+    (property "Footprint" "local:DSUB-15-HD_Female_Horizontal_P2.29x2.54mm_EdgePinOffset8.35mm_Housed_MountingHolesOffset10.89mm" (at 133.35 91.44 0)
       (effects (font (size 1.27 1.27)) hide)
     )
