File: vgaterm-io-faceboard/vgaterm-io-faceboard.kicad_sch (KiCad schematic)
At the start: 8 parts, among them J1 Conn_01x04, J1 USB_B_Micro UART, J2 Conn_01x02, J2 Conn_01x04

Commit message: current boards
Parts:
- added C1, C2, C3: C_Small, Capacitor_SMD:C_0805_2012Metric_Pad1.18x1.45mm_HandSolder, symbol Device:C_Small
- added R10, R7, R8, R9: R, Resistor_SMD:R_0805_2012Metric_Pad1.20x1.40mm_HandSolder, symbol Device:R
- added R17, R18: 27, Resistor_SMD:R_0805_2012Metric_Pad1.20x1.40mm_HandSolder, symbol Device:R_Small
- added R19: 4.7k, Resistor_SMD:R_0805_2012Metric_Pad1.20x1.40mm_HandSolder, symbol Device:R_Small
- added R20: 10k, Resistor_SMD:R_0805_2012Metric_Pad1.20x1.40mm_HandSolder, symbol Device:R_Small
- added U1: FT230XS, Package_SO:SSOP-16_3.9x4.9mm_P0.635mm, symbol Interface_USB:FT230XS
Connections:
- net D+: now also C1.1, R18.1; no longer J1.2 (Pin_2)
- net D-: now also C2.1, R17.1; no longer J1.3 (Pin_3)
- net GND: now also J2.1 (Pin_1), C1.2, C2.2, C3.2, R20.2, U1.13 (GND), U1.5 (GND); no longer J2.4 (Pin_4)
- net RXI_{0}: now also R8.2, U1.4 (RXD); no longer J2.1 (Pin_1), J2.3 (Pin_3)
- net S_{1}: now also J2.4 (Pin_4); no longer J2.1 (Pin_1)
- net TXI_{0}: now also R7.1, U1.1 (TXD); no longer J2.2 (Pin_2), J2.2 (Pin_2)
- net VCC: now also U1.12 (VCC); no longer J1.1 (VBUS)
- new net: J2.2 (Pin_2), R9.2
- new net: J1.2 (Pin_2), R7.2
- new net: J1.3 (Pin_3), R8.1
- new net: J1.1 (VBUS), R19.1
- new net: J2.3 (Pin_3), R10.1
- new net: U1.2 (~{RTS}), U1.6 (~{CTS})
- new net: R18.2, U1.8 (USBDP)
- new net: R17.2, U1.9 (USBDM)
- new net 3v3: C3.1, U1.10 (3V3OUT), U1.11 (~{RESET}), U1.3 (VCCIO)
- new net RXI_{1}: J2.1 (Pin_1), R10.2
- new net TXI_{1}: J2.2 (Pin_2), R9.1
- new net V_sense: R19.2, R20.1, U1.15 (CBUS0)
Other:
- moved on the sheet: D1, D2, J1, J2, R17, R18
